Commit message: gz bridge implementation: loaded lidar sensors, optimizing the world and rviz settings

File: spawn_robot/model/formula/urdf/formula_description.urdf.xacro (robot description, xacro)
@@ -1,5 +1,5 @@
 <?xml version="1.0"?>
 <robot xmlns:xacro="http://www.ros.org/wiki/xacro" name="formula">
-    <xacro:arg name="gpu" default="false"/>
+    <xacro:arg name="gpu" default="true"/>
     <xacro:property name="gpu" value="$(arg gpu)" />
     <xacro:arg name="organize_cloud" default="false"/>
@@ -12,6 +12,6 @@
     <xacro:include filename="$(find spawn_robot)/model/formula/urdf/vehicle_properties.urdf.xacro"/>
     <xacro:include filename="$(find spawn_robot)/model/formula/urdf/formula.gazebo"/>
-    <!-- <xacro:include filename="$(find spawn_robot)/model/formula/urdf/sensors/camera.urdf.xacro"/>
-    <xacro:include filename="$(find spawn_robot)/model/formula/urdf/sensors/vlp-16.urdf.xacro"/> -->
+    <!-- <xacro:include filename="$(find spawn_robot)/model/formula/urdf/sensors/camera.urdf.xacro"/> -->
+    <xacro:include filename="$(find spawn_robot)/model/formula/urdf/sensors/vlp-16.urdf.xacro"/>
     <!-- *************** -->
     <!-- Robots Elements -->
@@ -22,3 +22,6 @@
     <xacro:Rear_Right_Wheel/>
     <xacro:Rear_Left_Wheel/>
+    <xacro:VLP-16 parent="chassis" name="velodyne" topic="/velodyne_points" organize_cloud="${organize_cloud}" hz="10" samples="440" gpu="${gpu}">
+      <origin xyz="0 0 ${car_height - 0.23}" rpy="0 0 0" />
+    </xacro:VLP-16>
 </robot>

File: spawn_robot/model/formula/urdf/sensors/vlp-16.urdf.xacro (robot description, xacro)
@@ -18,10 +18,10 @@
         <visual>
             <geometry>
-            <mesh filename="package://spawn_robot/model/formula/meshes/VLP16_base_1.dae" />
+            <mesh filename="file://$(find spawn_robot)/model/formula/meshes/VLP16_base_1.dae" />
             </geometry>
         </visual>
         <visual>
             <geometry>
-            <mesh filename="package://spawn_robot/model/formula/meshes/VLP16_base_2.dae" />
+            <mesh filename="file://$(find spawn_robot)/model/formula/meshes/VLP16_base_2.dae" />
             </geometry>
         </visual>
@@ -47,5 +47,5 @@
             <origin xyz="0 0 -0.0377" />
             <geometry>
-            <mesh filename="package://spawn_robot/model/formula/meshes/VLP16_scan.dae" />
+            <mesh filename="file://$(find spawn_robot)/model/formula/meshes/VLP16_scan.dae" />
             </geometry>
         </visual>
@@ -56,12 +56,14 @@
         </collision>
         </link>
-        <!-- Gazebo requires the velodyne_gazebo_plugins package -->
         <gazebo reference="${name}">
         <xacro:if value="${gpu}">
-            <sensor type="gpu_ray" name="${name}-VLP16">
+            <sensor type="gpu_lidar" name="${name}-VLP16">
             <pose>0 0 0 0 0 0</pose>
-            <visualize>false</visualize>
+            <visualize>true</visualize>
             <update_rate>${hz}</update_rate>
-            <ray>
+            <always_on>1</always_on>
+            <topic>${topic}</topic>
+            <gz_frame_id>${name}</gz_frame_id>
+            <lidar>
                 <scan>
                 <horizontal>
@@ -88,56 +90,8 @@
                 <stddev>0.0</stddev>
                 </noise>
-            </ray>
-            <plugin name="gazebo_ros_laser_controller" filename="libgazebo_ros_velodyne_gpu_laser.so">
-                <topicName>${topic}</topicName>
-                <frameName>${name}</frameName>
-                <organize_cloud>${organize_cloud}</organize_cloud>
-                <min_range>${min_range}</min_range>
-                <max_range>${max_range}</max_range>
-                <gaussianNoise>${noise}</gaussianNoise>
-            </plugin>
+                <frame_id>${name}</frame_id>
+            </lidar>
             </sensor>
         </xacro:if>
-        <xacro:unless value="${gpu}">
-            <sensor type="ray" name="${name}-VLP16">
-            <pose>0 0 0 0 0 0</pose>
-            <visualize>false</visualize>
-            <update_rate>${hz}</update_rate>
-            <ray>
-                <scan>
-                <horizontal>
-                    <samples>${samples}</samples>
-                    <resolution>1</resolution>
-                    <min_angle>${min_angle}</min_angle>
-                    <max_angle>${max_angle}</max_angle>
-                </horizontal>
-                <vertical>
-                    <samples>${lasers}</samples>
-                    <resolution>1</resolution>
-                    <min_angle>-${15.0*M_PI/180.0}</min_angle>
-                    <max_angle> ${15.0*M_PI/180.0}</max_angle>
-                </vertical>
-                </scan>
-                <range>
-                <min>${collision_range}</min>
-                <max>${max_range+1}</max>
-                <resolution>0.001</resolution>
-                </range>
-                <noise>
-                <type>gaussian</type>
-                <mean>0.0</mean>
-                <stddev>0.0</stddev>
-                </noise>
-            </ray>
-            <plugin name="gazebo_ros_laser_controller" filename="libgazebo_ros_velodyne_laser.so">
-                <topicName>${topic}</topicName>
-                <frameName>${name}</frameName>
-                <organize_cloud>${organize_cloud}</organize_cloud>
-                <min_range>${min_range}</min_range>
-                <max_range>${max_range}</max_range>
-                <gaussianNoise>${noise}</gaussianNoise>
-            </plugin>
-            </sensor>
-        </xacro:unless>
         </gazebo>
     </xacro:macro>
